File: Projects/VF2/VF-2.kicad_sch (KiCad schematic)
At the start: 39 parts, among them P1 P, T1 MPSA42, T2 MPSA93, T3 IRF9540, T4 IRF540, U1 Opa2134, U2 OPA2134

Commit message: sch
Parts:
- renumbered T4 to T
Connections:
- net at C4.2, OUT., R13.1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: now also T.2 (D), T3.3 (S); no longer T. (S), T3. (S)
- net at D4.2 (A), R12.1, R6.1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: now also T.3 (S); no longer T. (S)
- net at D4.1 (K), D6.2 (A), T2. (E): now also T.1 (G); no longer T. (S)
- net at D3.1 (K), R5.2, R9.2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: now also T3.2 (D); no longer T3. (S)
- net at D3.2 (A), D5.1 (K), T1. (E): now also T3.1 (G); no longer T3. (S)

Commit message: sch-rajz-hiba-javitas
Connections:
- net at C4.2, OUT., R13.1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: now also T3.2 (D); no longer T3.3 (S)
- net at D3.1 (K), R5.2, R9.2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: now also T3.3 (S); no longer T3.2 (D)
Changed lines of the file:
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@@
 	(polyline
 		(pts
-			(xy -218.44 -10.16) (xy -19.05 -10.16)
+			(xy -223.52 1.27) (xy -24.13 1.27)
 		)
 		(stroke
@@
 	(polyline
 		(pts
-			(xy -218.44 125.73) (xy -19.05 125.73)
+			(xy -223.52 137.16) (xy -24.13 137.16)
 		)
 		(stroke
@@
 	(polyline
 		(pts
-			(xy -19.05 -10.16) (xy -19.05 125.73)
+			(xy -24.13 1.27) (xy -24.13 137.16)
 		)
 		(stroke
@@
 	(polyline
 		(pts
-			(xy -218.44 -10.16) (xy -218.44 125.73)
+			(xy -223.52 1.27) (xy -223.52 137.16)
 		)
 		(stroke
@@
 		(lib_id "Transistor_FET:IRF9540N")
 		(at 196.85 63.5 0)
+		(mirror x)
 		(unit 1)
 		(body_style 1)
@@
 		(in_pos_files yes)
 		(dnp no)
-		(fields_autoplaced yes)
 		(property "Reference" "T3"
-			(at 204.47 62.2299 0)
+			(at 204.47 64.7701 0)
 			(show_name no)
 			(do_not_autoplace no)
@@
 		)
 		(property "Value" "IRF9540"
-			(at 204.47 64.7699 0)
+			(at 204.47 62.2301 0)
 			(show_name no)
 			(do_not_autoplace no)
@@
 		)
 		(property "Footprint" "Package_TO_SOT_THT:TO-220-3_Vertical"
-			(at 201.93 65.405 0)
+			(at 201.93 61.595 0)
 			(hide yes)
 			(show_name no)
@@
 		)
 		(property "Datasheet" "http://www.irf.com/product-info/datasheets/data/irf9540n.pdf"
-			(at 201.93 67.31 0)
+			(at 201.93 59.69 0)
 			(hide yes)
 			(show_name no)
@@
 		)
 		(property "Description" "-23A Id, -100V Vds, 117mOhm Rds, P-Channel HEXFET Power MOSFET, TO-220"
-			(at 192.786 55.372 0)
-			(hide yes)
-			(show_name no)
+			(at 192.786 71.628 0)
+			(hide yes)
+			(show_name no)

Commit message: sch_javitas
Parts:
- removed T: IRF540, Package_TO_SOT_THT:TO-220-3_Vertical, symbol 000_Device:N_Channel_FET
- removed T3: IRF9540, Package_TO_SOT_THT:TO-220-3_Vertical, symbol Transistor_FET:IRF9540N
- added T3: IRF9540, Package_TO_SOT_THT:TO-220-3_Vertical, symbol 000_Device:Transistor_FET_P
- added T4: IRF540, Package_TO_SOT_THT:TO-220-3_Vertical, symbol 000_Device:Transistor_FET_P
- C1: value 1-10uF tantál -> 1-10uF tantál, ESR
- renumbered R6 to R6*
Connections:
- net at C4.2, OUT., R13.1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: now also T3.2 (D), T4.2 (D)
- net at D4.2 (A), R12.1, R6*.1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: now also T4.3 (S)
- net at D4.1 (K), D6.2 (A), T2. (E): now also T4.1 (G)
- net at D3.1 (K), R5.2, R9.2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: now also T3.3 (S)
- net at D3.2 (A), D5.1 (K), T1. (E): now also T3.1 (G)
Other:
- moved on the sheet: C2, C4, R3, R4

Commit message: sch
Parts:
- C1: value 1-10uF tantál, ESR -> 1uF MKP
- P1: value P -> 2k2
- R5: value 2k2 * -> 1k8 *
- R6: renamed from R6*; value 2k2* -> 1k8*
Other:
- note added: "3mA"

Commit message: 20261008
Parts:
- C2, C3, C4, C5, C6, C7, C8, R3, R4, R7, R8: footprint Package_SO:SOIC-8_3.9x4.9mm_P1.27mm -> (none)
- D1, D2, D3, D4, IN1: footprint Diode_SMD:Littelfuse_PolyZen-LS -> (none)
- D5, D6, P1, Vcc2: footprint Diode_THT:D_DO-35_SOD27_P7.62mm_Horizontal -> (none)
- OUT1: renamed from OUT; footprint Diode_SMD:Littelfuse_PolyZen-LS -> (none)
- T1, T2: footprint Package_TO_SOT_THT:TO-92_Inline -> (none)
- T3, T4: footprint Package_TO_SOT_THT:TO-220-3_Vertical -> (none)
Changed lines of the file:
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@@
 			)
 		)
-		(property "Footprint" "Package_SO:SOIC-8_3.9x4.9mm_P1.27mm"
+		(property "Footprint" ""
 			(at 154.94 74.168 90)
 			(hide yes)
@@
 		(in_pos_files yes)
 		(dnp no)
-		(property "Reference" "OUT"
+		(property "Reference" "OUT1"
 			(at 228.6 93.98 0)
 			(show_name no)
@@
 			)
 		)
-		(property "Footprint" "Diode_SMD:Littelfuse_PolyZen-LS"
+		(property "Footprint" ""
 			(at 224.282 96.266 0)
 			(hide yes)
@@
 			(project "VF-2"
 				(path "/a4dac9d1-a4ef-4cb2-9f5b-b3d5cd44301f"
-					(reference "OUT")
+					(reference "OUT1")
 					(unit 1)
 				)
@@
 			)
 		)
-		(property "Footprint" "Diode_THT:D_DO-35_SOD27_P7.62mm_Horizontal"
+		(property "Footprint" ""
 			(at 177.038 98.044 90)
 			(hide yes)
@@
 			)
 		)
-		(property "Footprint" "Package_SO:SOIC-8_3.9x4.9mm_P1.27mm"
+		(property "Footprint" ""
 			(at 78.74 174.9552 0)
 			(hide yes)
@@
 			)
 		)
-		(property "Footprint" "Package_TO_SOT_THT:TO-220-3_Vertical"
+		(property "Footprint" ""
 			(at 200.66 61.595 0)
 			(hide yes)
@@
 			)
 		)
-		(property "Footprint" "Package_SO:SOIC-8_3.9x4.9mm_P1.27mm"
+		(property "Footprint" ""
 			(at 160.9852 86.36 0)
 			(hide yes)
@@
 			)
 		)
-		(property "Footprint" "Package_TO_SOT_THT:TO-92_Inline"
+		(property "Footprint" ""
 			(at 187.706 139.7 0)
 			(hide yes)
@@
 			)
 		)
-		(property "Footprint" "Diode_THT:D_DO-35_SOD27_P7.62mm_Horizontal"
+		(property "Footprint" ""
 			(at 186.436 149.352 0)
 			(hide yes)
@@
 			)
 		)
-		(property "Footprint" "Package_SO:SOIC-8_3.9x4.9mm_P1.27mm"
+		(property "Footprint" ""
 			(at 98.7552 101.6 0)
 			(hide yes)
@@
 			)
 		)
-		(property "Footprint" "Diode_SMD:Littelfuse_PolyZen-LS"
+		(property "Footprint" ""
 			(at 66.04 90.17 0)
 			(hide yes)
@@
 			)
 		)
-		(property "Footprint" "Package_SO:SOIC-8_3.9x4.9mm_P1.27mm"
+		(property "Footprint" ""
 			(at 97.79 175.768 90)
 			(hide yes)
@@
 			)
 		)
-		(property "Footprint" "Diode_THT:D_DO-35_SOD27_P7.62mm_Horizontal"
+		(property "Footprint" ""
 			(at 186.436 59.182 0)
 			(hide yes)
@@
 			)
 		)
-		(property "Footprint" "Diode_SMD:Littelfuse_PolyZen-LS"
+		(property "Footprint" ""
 			(at 168.148 44.45 0)
 			(hide yes)
@@
 			)
 		)
-		(property "Footprint" "Package_SO:SOIC-8_3.9x4.9mm_P1.27mm"
+		(property "Footprint" ""
 			(at 154.94 133.858 90)
 			(hide yes)
@@
 			)
 		)
-		(property "Footprint" "Package_SO:SOIC-8_3.9x4.9mm_P1.27mm"
+		(property "Footprint" ""
 			(at 127.9652 114.3 0)
 			(hide yes)
@@
 			)
 		)
-		(property "Footprint" "Package_TO_SOT_THT:TO-92_Inline"
+		(property "Footprint" ""
 			(at 187.706 80.01 0)
 			(hide yes)
@@
 			)
 		)
-		(property "Footprint" "Package_SO:SOIC-8_3.9x4.9mm_P1.27mm"
+		(property "Footprint" ""
 			(at 123.19 160.3248 0)
 			(hide yes)
@@
 			)
 		)
-		(property "Footprint" "Diode_SMD:Littelfuse_PolyZen-LS"
+		(property "Footprint" ""
 			(at 138.938 82.55 0)
 			(hide yes)
@@
 			)
 		)
-		(property "Footprint" "Package_SO:SOIC-8_3.9x4.9mm_P1.27mm"
+		(property "Footprint" ""
 			(at 160.9852 114.3 0)
 			(hide yes)
@@
 			)
 		)
-		(property "Footprint" "Diode_SMD:Littelfuse_PolyZen-LS"
+		(property "Footprint" ""
 			(at 138.938 110.49 0)
 			(hide yes)
@@
 			)
 		)
-		(property "Footprint" "Package_SO:SOIC-8_3.9x4.9mm_P1.27mm"
+		(property "Footprint" ""
 			(at 121.92 175.768 90)
 			(hide yes)
@@
 			)
 		)
-		(property "Footprint" "Diode_SMD:Littelfuse_PolyZen-LS"
+		(property "Footprint" ""
 			(at 169.418 161.29 0)
 			(hide yes)
@@
 			)
 		)
-		(property "Footprint" "Diode_THT:D_DO-35_SOD27_P7.62mm_Horizontal"
+		(property "Footprint" ""
 			(at 219.71 168.91 0)
 			(hide yes)
@@
 			)
 		)
-		(property "Footprint" "Package_TO_SOT_THT:TO-220-3_Vertical"
+		(property "Footprint" ""
 			(at 200.66 147.066 0)
 			(hide yes)
@@
 			)
 		)
-		(property "Footprint" "Package_SO:SOIC-8_3.9x4.9mm_P1.27mm"
+		(property "Footprint" ""
 			(at 127.9652 86.36 0)
 			(hide yes)

Commit message: 2
Parts:
- added R14, R15: 100R, symbol 000_Device:R
Connections:
- net at D3.2 (A), D5.1 (K), T1. (E): now also R14.2; no longer T3.1 (G)
- net at D4.1 (K), D6.2 (A), T2. (E): now also R15.2; no longer T4.1 (G)
- new net: R15.1, T4.1 (G)
- new net: R14.1, T3.1 (G)
Other:
- moved on the sheet: T3, T4

Commit message: 1
Parts:
- R14, R15: value 100R -> 220R
Changed lines of the file:
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@@
 			)
 		)
-		(property "Value" "100R"
+		(property "Value" "220R"
 			(at 196.85 138.43 90)
 			(show_name no)
@@
 			)
 		)
-		(property "Value" "100R"
+		(property "Value" "220R"
 			(at 194.31 60.96 90)
 			(show_name no)

Commit message: 2
Parts:
- R14, R15: value 220R -> 100R
Changed lines of the file:
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@@
 			)
 		)
-		(property "Value" "220R"
+		(property "Value" "100R"
 			(at 196.85 138.43 90)
 			(show_name no)
@@
 			)
 		)
-		(property "Value" "220R"
+		(property "Value" "100R"
 			(at 194.31 60.96 90)
 			(show_name no)
