File: Projects/VF2/VF-2-modositott.kicad_sch (KiCad schematic)
At the start: 39 parts, among them T1 MPSA42, T2 MPSA93, T3 IRF9540, T4 IRF540, U1 Opa2134, U2 OPA2134

Commit message: sch
Parts:
- removed D1: ZPD12, Diode_SMD:Littelfuse_PolyZen-LS, symbol Device:D_Zener
- removed IN: (no value), Diode_SMD:Littelfuse_PolyZen-LS, symbol 001_atmeneti_Device:Vcc
- removed P: P, Diode_THT:D_DO-35_SOD27_P7.62mm_Horizontal, symbol Device:R_Trim
- added D1: ZPD12, Diode_SMD:Littelfuse_PolyZen-LS, symbol 000_Device:D_Zener
- added IN1: (no value), Diode_SMD:Littelfuse_PolyZen-LS, symbol 001_atmeneti_Device:Vcc
- added P1: P, Diode_THT:D_DO-35_SOD27_P7.62mm_Horizontal, symbol Device:R_Trim
Connections:
- net GND: now also D1.2 (A)
- net at R11.2: now also P1., P1.2
- net at R10.1, R13.2, U1.1: now also P1.1
- net at C5.1, R5.1, R8.2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: now also D1.1 (K)
- net at C1.1: now also IN1.
Other:
- note added: "VF2"
- company: (none) -> Nautilus Művek
