File: Projects/Sablon.kicad_sch (KiCad schematic)
At the start: 4 parts

Commit message: sch
Changed lines of the file:
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@@
 	(polyline
 		(pts
-			(xy -33.02 254) (xy -177.8 254)
+			(xy -40.64 248.92) (xy -185.42 248.92)
 		)
 		(stroke
@@
 	(polyline
 		(pts
-			(xy -33.02 153.67) (xy -33.02 254)
+			(xy -40.64 148.59) (xy -40.64 248.92)
 		)
 		(stroke
@@
 	(polyline
 		(pts
-			(xy -177.8 153.67) (xy -177.8 254)
+			(xy -185.42 148.59) (xy -185.42 248.92)
 		)
 		(stroke
@@
 	(polyline
 		(pts
-			(xy -177.8 153.67) (xy -33.02 153.67)
+			(xy -185.42 148.59) (xy -40.64 148.59)
 		)
 		(stroke
