File: Projects/VF2_ver_6_0/VF2_ver_6_0.kicad_sch (KiCad schematic)
At the start: 2 parts

Commit message: sch
Parts:
- removed R? (x2): R, symbol Device:R
- added R: R, symbol Device:R
- added R?: R, symbol 000_Small_Device:R
Changed lines of the file:
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@@
 (kicad_sch (version 20211123) (generator eeschema)
   (paper "A4")
-  (polyline (pts (xy 0 0) (xy 0 149.86))
-    (stroke (width 0) (type default) (color 0 0 0 0))
-  )
-  (polyline (pts (xy 210.82 149.86) (xy 210.82 0))
-    (stroke (width 0) (type default) (color 0 0 0 0))
-  )
-  (polyline (pts (xy 0 149.86) (xy 210.82 149.86))
-    (stroke (width 0) (type default) (color 0 0 0 0))
-  )
-  (polyline (pts (xy 0 0) (xy 210.82 0))
-    (stroke (width 0) (type default) (color 0 0 0 0))
-  )
-  (symbol (lib_name "R_1") (lib_id "Device:R") (at 69.85 33.02 0) (unit 1)
+  (symbol (lib_id "000_Small_Device:R") (at 100.33 85.09 0) (unit 1)
     (in_bom yes) (on_board yes) (fields_autoplaced)
-    (property "Reference" "R?" (id 0) (at 72.39 31.7499 0)
-      (effects (font (size 1.27 1.27)) (justify left))
+    (property "Reference" "R?" (id 0) (at 102.87 83.82 0)
+      (effects (font (size 1.4 1.4)) (justify left))
     )
-    (property "Value" "R" (id 1) (at 72.39 34.2899 0)
-      (effects (font (size 1.27 1.27)) (justify left))
+    (property "Value" "R" (id 1) (at 102.87 86.36 0)
+      (effects (font (size 1.4 1.4)) (justify left))
     )
-    (property "Footprint" "" (id 2) (at 68.072 33.02 90)
+    (property "Footprint" "" (id 2) (at 98.552 85.09 90)
       (effects (font (size 1.27 1.27)) hide)
     )
-    (property "Datasheet" "~" (id 3) (at 69.85 33.02 0)
+    (property "Datasheet" "~" (id 3) (at 100.33 85.09 0)
       (effects (font (size 1.27 1.27)) hide)
     )
@@
     (pin "2")
   )
-  (symbol (lib_id "Device:R") (at 69.85 50.8 0) (unit 1)
+  (symbol (lib_id "Device:R") (at 77.47 82.55 0) (unit 1)
     (in_bom yes) (on_board yes) (fields_autoplaced)
-    (property "Reference" "R?" (id 0) (at 72.39 49.5299 0)
-      (effects (font (size 1.27 1.27)) (justify left))
+    (property "Reference" "R" (id 0) (at 80.01 81.2799 0)
+      (effects (font (size 1.4 1.4)) (justify left))
     )
-    (property "Value" "R" (id 1) (at 72.39 52.0699 0)
-      (effects (font (size 1.27 1.27)) (justify left))
+    (property "Value" "R" (id 1) (at 80.01 83.8199 0)
+      (effects (font (size 1.4 1.4)) (justify left))
     )
-    (property "Footprint" "" (id 2) (at 68.072 50.8 90)
+    (property "Footprint" "" (id 2) (at 75.692 82.55 90)
       (effects (font (size 1.27 1.27)) hide)
     )
-    (property "Datasheet" "~" (id 3) (at 69.85 50.8 0)
+    (property "Datasheet" "~" (id 3) (at 77.47 82.55 0)
       (effects (font (size 1.27 1.27)) hide)
     )
@@
   )
   (symbol_instances
-    (path "/25eeb5a3-4108-4450-9596-f4d1a9d9a4db"
+    (path "/9c480b29-c87d-4b36-b810-8c82dce65a46"
+      (reference "R") (unit 1) (value "R") (footprint "")
+    )
+    (path "/8f1d8454-16bf-4071-a8dc-4bf2a7a3cdd2"
       (reference "R?") (unit 1) (value "R") (footprint "")
     )
-    (path "/4238c926-29b5-4dc6-ace6-dc3fd335cf31"
-      (reference "R?") (unit 1) (value "R") (footprint "")
-    )
