File: Projects/HIRAGA/HIRAGA.kicad_sch (KiCad schematic)
At the start: 4 parts

Commit message: sch
Parts:
- removed C2: C_Polarized, Package_SO:SOIC-8_3.9x4.9mm_P1.27mm, symbol 000_Device:C_Polarized
- removed C3: 600pF, Package_SO:SOIC-8_3.9x4.9mm_P1.27mm, symbol Device:C
- removed D2: D, symbol Device:D
- removed R1: 5k6, Package_DIP:DIP-8_W7.62mm, symbol 000_Small_Device:R
