File: Projects/Conductor-V2/Conductor-V2.kicad_sch (KiCad schematic)
At the start: 23 parts, among them T1 FET_N, T2 FET_P, U1 OPA2134

Commit message: x
Parts:
- removed T1: FET_N, Package_TO_SOT_THT:TO-220-3_Vertical, symbol 000_Small_Device:Transistor_FET_N
- removed T2: FET_P, Package_TO_SOT_THT:TO-220-3_Vertical, symbol 000_Small_Device:Transistor_FET_P
- removed unit 3 of U1
- added D1, D2: TL431, symbol 000_Small_Device:TL431D
- added D3, D5: 10V, symbol Device:D_Zener
- added D4, D6: 1N4148, symbol Device:D
- added R10: 2k7, symbol 000_Small_Device:R
- added R11: 11k, symbol 000_Small_Device:R
- added R12, R15: 820R, symbol 000_Small_Device:R
- added R13, R21: 220R, symbol 000_Small_Device:R
- added R14: 18k, symbol 000_Small_Device:R
- added R16, R9: 1k5, symbol 000_Small_Device:R
- added R17: 4k3, symbol 000_Small_Device:R
- added R19, R20: R, symbol 000_Small_Device:R
- added T1: MPSA42, symbol 000_Small_Device:Transistor_NPN_EBC
- added T2: MPSA92, symbol 000_Small_Device:Transistor_PNP_EBC
- added T3: IRF9540, Package_TO_SOT_THT:TO-220-3_Vertical, symbol 000_Small_Device:Transistor_FET_P
- added T4: FET_N, Package_TO_SOT_THT:TO-220-3_Vertical, symbol 000_Small_Device:Transistor_FET_N
- added U2: OPA2134, symbol Amplifier_Operational:OPA2134
- C4: value C -> 39p
- C5: value C_P -> 100uF
- C6: value C_P -> 100nF
- R3: value R -> 1k
- R5: value R -> 33k
- R6: value R -> 11k
- R7: renamed from R6; value R -> 22k
- R8: renamed from R7; value R -> 4k3
- renumbered R8 to R18
Connections:
- net GNDD: now also C5.2, C6.1, R3.1, D1.[2,3,6,7] (A), D2.1 (K), R20.1
- net at U1.1: now also R8.1, R10.2, R11.1
- net at C4.1, R5.2: now also OUT., R11.2, T3.2 (D), T4.2 (D)
- net at VCC.: now also D6.1 (K), R16.2, T4.3 (S)
- net at R7.1: now also D2.8 (REF), R17.2
- net at R7.2: now also C6.2, D2.[2,3,6,7] (A), R14.2, R16.1, T2.2 (B), U2.4 (V-)
- net at R8.2: now also T2.1 (E)
- net at C5.1: now also R6.1, D1.1 (K), R9.1, T1.2 (B)
- net at R6.2: now also D1.8 (REF), R14.1
- net at R18.: now also R18.2, R17.1
- net at R18.1: now also R19.2
- net at VCC.: now also D4.2 (A), R9.2, T3.3 (S)
- new net: D3.2 (A), R12.2, R13.1, T1.3 (C)
- new net: R13.2, T3.1 (G)
- new net: R21.2, T4.1 (G)
- new net: D5.1 (K), R15.1, R21.1, T2.3 (C)
- new net: D5.2 (A), D6.2 (A), R15.2
- new net: D3.1 (K), D4.1 (K), R12.1
- new net: R10.1, T1.1 (E)
- new net: R19.1, R20.2
Other:
- moved on the sheet: C1, C2, C3, C4, C5, C6, GND, IN, OUT, R1, R18, R2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

Commit message: x
Parts:
- added T5: BD139, symbol 000_Small_Device:Transistor_NPN_EBC
- C3: value C -> 330nF
- R18: value R_Trim -> 2k2
- R19: value R -> 560R
- R20: value R -> 15k
- T4: value FET_N -> IRF540
Connections:
- net GNDD: now also T5.3 (C)
- net at U2.8 (V+): now also C5.1, D1.1 (K), R6.1, R9.1, T1.2 (B)
- net at R19.1, R20.2: now also T5.2 (B)
- net at R17.1, R18., R18.2: now also T5.1 (E)
Other:
- moved on the sheet: R14, R18, R19, R20, R6

Commit message: 1
Parts:
- R11: value 11k -> 10k
- R14: value 18k -> 15k
- R16: value 1k5 -> 1k2
- R6: value 11k -> 8k6
- R7: value 22k -> 2k2
Changed lines of the file:
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@@
 			)
 		)
-		(property "Value" "11k"
+		(property "Value" "10k"
 			(at 172.72 90.17 90)
 			(show_name no)
@@
 			)
 		)
-		(property "Value" "18k"
+		(property "Value" "15k"
 			(at 138.43 101.6 0)
 			(show_name no)
@@
 		(in_pos_files yes)
 		(dnp no)
-		(fields_autoplaced yes)
 		(property "Reference" "R19"
-			(at 111.7601 137.16 0)
+			(at 106.68 129.54 90)
 			(show_name no)
 			(do_not_autoplace no)
@@
 		)
 		(property "Value" "560R"
-			(at 109.2201 137.16 0)
+			(at 106.68 132.08 90)
 			(show_name no)
 			(do_not_autoplace no)
@@
 			)
 		)
-		(property "Value" "22k"
+		(property "Value" "2k2"
 			(at 149.86 114.3 0)
 			(show_name no)
@@
 			)
 		)
-		(property "Value" "1k5"
+		(property "Value" "1k2"
 			(at 161.29 147.32 90)
 			(show_name no)
@@
 		(in_pos_files yes)
 		(dnp no)
-		(fields_autoplaced yes)
 		(property "Reference" "R6"
-			(at 147.32 71.1199 0)
-			(show_name no)
-			(do_not_autoplace no)
-			(effects
-				(font
-					(size 1.27 1.27)
-				)
-				(justify left)
-			)
-		)
-		(property "Value" "11k"
-			(at 147.32 73.6599 0)
+			(at 146.459 70.9478 0)
+			(show_name no)
+			(do_not_autoplace no)
+			(effects
+				(font
+					(size 1.27 1.27)
+				)
+				(justify left)
+			)
+		)
+		(property "Value" "8k6"
+			(at 146.2868 73.2724 0)
 			(show_name no)
 			(do_not_autoplace no)
@@
 		)
 		(property "Value" "2k2"
-			(at 118.11 132.08 90)
+			(at 119.38 139.7 90)
 			(show_name no)
 			(do_not_autoplace no)
@@
 		(in_pos_files yes)
 		(dnp no)
-		(fields_autoplaced yes)
 		(property "Reference" "R20"
-			(at 100.3301 137.16 0)
+			(at 96.52 129.54 90)
 			(show_name no)
 			(do_not_autoplace no)
@@
 		)
 		(property "Value" "15k"
-			(at 97.7901 137.16 0)
-			(show_name no)
-			(do_not_autoplace no)
+			(at 96.52 132.08 90)
+			(show_name no)
+			(do_not_autoplace no)

Commit message: 2
Parts:
- added R6B, R6C: 220R, symbol 000_Small_Device:R
- R6: value 8k6 -> 8k2
Connections:
- net at D1.8 (REF), R14.1: now also R6C.1; no longer R6.2
- new net: R6B.2, R6C.2
- new net: R6.2, R6B.1
Other:
- note added: "R6, R6B, R6C: 8k6 helyett van, azt nem tudtam venni."
- moved on the sheet: D1, R14, R6
