File: Projects/ConductorV2/ConductorV2.kicad_sch (KiCad schematic)
At the start: 47 parts, among them T1 MPSA42, T2 MPSA92, T3 IRF9540, T4 IRF540, T5 BD139, U1 OPA2134, U2 OPA2134

Commit message: v
Parts:
- R16: value 1k2 -> 1k5
Other:
- note added: "10 mA"
- note added: "10mA"

Commit message: 1
Parts:
- R10: value 2k7 -> 2k7 vagy 4k3 ?
- renumbered R6 to R6A
Connections:
- net at C3.2, R3.2, R4.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: now also C4.1, R5.2; no longer C4.2, R5.1
- net at OUT., R11.2, T3.2 (D)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: now also C4.2, R5.1; no longer C4.1, R5.2
Other:
- note removed: "R6, R6B, R6C: 8k6 helyett van, azt nem tudtam venni."
- moved on the sheet: C3, C4, D1, R14, R2, R3, R4, R5, R6A, R6B, R6C, R7

Commit message: x
Other:
- note added: "ConductorV2 amplifier"
Changed lines of the file:
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@@
 		)
 	)
+	(text "ConductorV2 amplifier"
+		(exclude_from_sim no)
+		(at 137.16 54.61 0)
+		(effects
+			(font
+				(size 2 2)
+			)
+		)
+	)
 	(text "10mA"
 		(exclude_from_sim no)
@@
 	)
 	(junction
-		(at 205.74 149.86)
-		(diameter 0)
-		(color 0 0 0 0)
-	)
-	(junction
 		(at 153.67 66.04)
 		(diameter 0)
@@
 	(wire
 		(pts
-			(xy 86.36 101.6) (xy 86.36 102.87)
-		)
-		(stroke
-			(width 0)
-			(type default)
-		)
-	)
-	(wire
-		(pts
 			(xy 123.19 134.62) (xy 130.81 134.62)
 		)
@@
 	(wire
 		(pts
-			(xy 205.74 149.86) (xy 201.93 149.86)
-		)
-		(stroke
-			(width 0)
-			(type default)
-		)
-	)
-	(wire
-		(pts
 			(xy 148.59 119.38) (xy 154.94 119.38)
 		)
@@
 		)
 	)
+	(wire
+		(pts
+			(xy 201.93 149.86) (xy 205.74 149.86)
+		)
+		(stroke
+			(width 0)
+			(type default)
+		)
+	)
 	(polyline
 		(pts
@@
 	(symbol
 		(lib_id "power:PWR_FLAG")
-		(at 205.74 149.86 180)
+		(at 201.93 149.86 180)
 		(unit 1)
 		(body_style 1)
@@
 		(fields_autoplaced yes)
 		(property "Reference" "#FLG01"
-			(at 205.74 151.765 0)
+			(at 201.93 151.765 0)
 			(hide yes)
 			(show_name no)
@@
 		)
 		(property "Value" "PWR_FLAG"
-			(at 205.74 154.94 0)
+			(at 201.93 154.94 0)
 			(hide yes)
 			(show_name no)
@@
 		)
 		(property "Footprint" ""
-			(at 205.74 149.86 0)
+			(at 201.93 149.86 0)
 			(hide yes)
 			(show_name no)
@@
 		)
 		(property "Datasheet" ""
-			(at 205.74 149.86 0)
+			(at 201.93 149.86 0)
 			(hide yes)
 			(show_name no)
@@
 		)
 		(property "Description" "Special symbol for telling ERC where power comes from"
-			(at 205.74 149.86 0)
+			(at 201.93 149.86 0)
 			(hide yes)
 			(show_name no)
@@
 	(symbol
 		(lib_id "power:PWR_FLAG")
-		(at 86.36 101.6 0)
+		(at 86.36 102.87 0)
 		(unit 1)
 		(body_style 1)
@@
 		(fields_autoplaced yes)
 		(property "Reference" "#FLG03"
-			(at 86.36 99.695 0)
+			(at 86.36 100.965 0)
 			(hide yes)
 			(show_name no)
@@
 		)
 		(property "Value" "PWR_FLAG"
-			(at 86.36 96.52 0)
+			(at 86.36 97.79 0)
 			(hide yes)
 			(show_name no)
@@
 		)
 		(property "Footprint" ""
-			(at 86.36 101.6 0)
+			(at 86.36 102.87 0)
 			(hide yes)
 			(show_name no)
@@
 		)
 		(property "Datasheet" ""
-			(at 86.36 101.6 0)
+			(at 86.36 102.87 0)
 			(hide yes)
 			(show_name no)
@@
 		)
 		(property "Description" "Special symbol for telling ERC where power comes from"
-			(at 86.36 101.6 0)
+			(at 86.36 102.87 0)
 			(hide yes)
 			(show_name no)
