File: Projects/ZaborszkyVedelem/ZaborszkyVedelem.kicad_sch (KiCad schematic)
At the start: 1 part, among them K2 kapcsolo

Commit message: conductor-sch
Parts:
- added C1, C2: C, symbol 000_Small_Device:C
- added T1, T2: Transistor_NPN_EBC, symbol 000_Small_Device:Transistor_NPN_EBC
- added T3: Transistor_PNP_EBC, symbol 000_Small_Device:Transistor_PNP_EBC

Commit message: 2
Connections:
- net at T1.2 (B): now also T2.1 (E)
- net at T1.3 (C): now also T3.1 (E)
- net at T3.2 (B): now also T2.3 (C)
Other:
- moved on the sheet: T1, T2, T3
Changed lines of the file:
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@@
 	(generator_version "10.0")
 	(paper "A4")
+	(wire
+		(pts
+			(xy 93.98 91.44) (xy 99.06 91.44)
+		)
+		(stroke
+			(width 0)
+			(type default)
+		)
+	)
 	(polyline
 		(pts
@@
 		)
 	)
+	(wire
+		(pts
+			(xy 86.36 106.68) (xy 86.36 96.52)
+		)
+		(stroke
+			(width 0)
+			(type default)
+		)
+	)
 	(polyline
 		(pts
@@
 		)
 	)
+	(wire
+		(pts
+			(xy 109.22 106.68) (xy 86.36 106.68)
+		)
+		(stroke
+			(width 0)
+			(type default)
+		)
+	)
 	(polyline
 		(pts
@@
 		(pts
 			(xy 48.26 38.1) (xy 48.26 173.99)
+		)
+		(stroke
+			(width 0)
+			(type default)
+		)
+	)
+	(wire
+		(pts
+			(xy 109.22 96.52) (xy 106.68 96.52)
 		)
 		(stroke
@@
 	(symbol
 		(lib_id "000_Small_Device:Transistor_NPN_EBC")
-		(at 90 97 0)
+		(at 91.44 96.52 0)
 		(unit 1)
 		(body_style 1)
@@
 		(in_pos_files yes)
 		(dnp no)
-		(fields_autoplaced yes)
 		(property "Reference" "T1"
-			(at 95.73 95.7299 0)
+			(at 83.82 93.98 0)
 			(show_name no)
 			(do_not_autoplace no)
@@
 		)
 		(property "Value" "Transistor_NPN_EBC"
-			(at 95.73 98.2699 0)
+			(at 85.09 104.14 0)
 			(show_name no)
 			(do_not_autoplace no)
@@
 		)
 		(property "Footprint" ""
-			(at 95.08 94.46 0)
+			(at 96.52 93.98 0)
 			(hide yes)
 			(show_name no)
@@
 		)
 		(property "Datasheet" ""
-			(at 90 97 0)
+			(at 91.44 96.52 0)
 			(hide yes)
 			(show_name no)
@@
 		)
 		(property "Description" "NPN transistor, emitter/base/collector"
-			(at 90 97 0)
+			(at 91.44 96.52 0)
 			(hide yes)
 			(show_name no)
@@
 		)
 		(property "Sim.Device" "NPN"
-			(at 90 97 0)
+			(at 91.44 96.52 0)
 			(hide yes)
 			(show_name no)
@@
 		)
 		(property "Sim.Pins" "1=E 2=B 3=C"
-			(at 90 97 0)
+			(at 91.44 96.52 0)
 			(hide yes)
 			(show_name no)
@@
 	(symbol
 		(lib_id "000_Small_Device:Transistor_PNP_EBC")
-		(at 113 93 0)
+		(at 101.6 96.52 180)
 		(unit 1)
 		(body_style 1)
@@
 		(in_pos_files yes)
 		(dnp no)
-		(fields_autoplaced yes)
 		(property "Reference" "T3"
-			(at 118.89 91.7299 0)
+			(at 104.14 91.44 0)
 			(show_name no)
 			(do_not_autoplace no)
@@
 		)
 		(property "Value" "Transistor_PNP_EBC"
-			(at 118.89 94.2699 0)
+			(at 109.22 87.63 0)
 			(show_name no)
 			(do_not_autoplace no)
@@
 		)
 		(property "Footprint" ""
-			(at 118.08 90.46 0)
+			(at 96.52 99.06 0)
 			(hide yes)
 			(show_name no)
@@
 		)
 		(property "Datasheet" ""
-			(at 113 93 0)
+			(at 101.6 96.52 0)
 			(hide yes)
 			(show_name no)
@@
 		)
 		(property "Description" "PNP transistor, emitter/base/collector"
-			(at 113 93 0)
+			(at 101.6 96.52 0)
 			(hide yes)
 			(show_name no)
@@
 		)
 		(property "Sim.Device" "PNP"
-			(at 113 93 0)
+			(at 101.6 96.52 0)
 			(hide yes)
 			(show_name no)
@@
 		)
 		(property "Sim.Pins" "1=E 2=B 3=C"
-			(at 113 93 0)
+			(at 101.6 96.52 0)
 			(hide yes)
 			(show_name no)
@@
 	(symbol
 		(lib_id "000_Small_Device:Transistor_NPN_EBC")
-		(at 105 105 0)
+		(at 111.76 101.6 0)
+		(mirror y)
 		(unit 1)
 		(body_style 1)
@@
 		(in_pos_files yes)
 		(dnp no)
-		(fields_autoplaced yes)
 		(property "Reference" "T2"
-			(at 110.46 103.7299 0)
+			(at 114.3 105.41 0)
 			(show_name no)
 			(do_not_autoplace no)
@@
 		)
 		(property "Value" "Transistor_NPN_EBC"
-			(at 110.46 106.2699 0)
+			(at 132.08 96.52 0)
 			(show_name no)
 			(do_not_autoplace no)
@@
 		)
 		(property "Footprint" ""
-			(at 110.08 102.46 0)
+			(at 106.68 99.06 0)
 			(hide yes)
 			(show_name no)
@@
 		)
 		(property "Datasheet" ""
-			(at 105 105 0)
+			(at 111.76 101.6 0)
 			(hide yes)
 			(show_name no)
@@
 		)
 		(property "Description" "NPN transistor, emitter/base/collector"
-			(at 105 105 0)
+			(at 111.76 101.6 0)
 			(hide yes)
 			(show_name no)
@@
 		)
 		(property "Sim.Device" "NPN"
-			(at 105 105 0)
+			(at 111.76 101.6 0)
 			(hide yes)
 			(show_name no)
@@
 		)
 		(property "Sim.Pins" "1=E 2=B 3=C"
-			(at 105 105 0)
-			(hide yes)
-			(show_name no)
+			(at 111.76 101.6 0)
+			(hide yes)
+			(show_name no)

Commit message: vedelem
Parts:
- removed K2: kapcsolo, 000_Button_Switch:SW_Simpla_Forrszemes, symbol 001_atmeneti_Device:kapcsolo
- added C3: 220uF, symbol 000_Small_Device:C_P
- added C4: 4,7uF Tantal, symbol 000_Small_Device:C_P
- added C5: 470nF, symbol 000_Small_Device:C
- added C6: 100pF, symbol 000_Small_Device:C
- added C7: 4,7uF Tantal, symbol 000_Small_Device:C
- added D1: 1N4148, symbol Device:D
- added D2, D3: 1N4001, symbol 000_Small_Device:D
- added D4, D5, D6: 1N4148, symbol 000_Small_Device:D
- added K1: SW_SPST, symbol Switch:SW_SPST
- added R1: 30k, symbol 000_Small_Device:R
- added R10, R11: 27k, symbol 000_Small_Device:R
- added R12, R14: 150k, symbol 000_Small_Device:R
- added R13: 1k, symbol 000_Small_Device:R
- added R15, R4, R5: 100k, symbol 000_Small_Device:R
- added R16, R6: 2k2, symbol 000_Small_Device:R
- added R17: 270R, symbol 000_Small_Device:R
- added R2: 68k, symbol 000_Small_Device:R
- added R3: 1M, symbol 000_Small_Device:R
- added R7: 220k, symbol 000_Small_Device:R
- added R8: ***, symbol 000_Small_Device:R
- added R9: 180k, symbol 000_Small_Device:R
- added Relé: G2RL-1A-E, Relay_THT:Relay_SPST_Omron_G2RL-1A-E, symbol Relay:G2RL-1A-E
- added T10, T11, T4, T6, T8, T9: BC238, symbol 000_Small_Device:Transistor_NPN_EBC
- added T5, T7: 2N2219, symbol 000_Small_Device:Transistor_NPN_EBC
- added Végfok: (no value), symbol 000_Small_Device:Csatlakozo
- C1: value C -> 2,2uF
- C2: value C -> 1uF
- T1, T2: value Transistor_NPN_EBC -> BC238
- T3: value Transistor_PNP_EBC -> BC214
Connections:
- net GNDD: now reaches T1.1 (E)
- net GNDD: now also C1.2, C2.2, T2.2 (B), T3.3 (C), C3.2, C5.2, D1.2 (A), D6.2 (A), K1.1 (A), R1.1, R13.2, R15.2, R3.2, R5.2, Relé.13, T5.1 (E), T7.1 (E), T8.1 (E), T9.1 (E), Végfok.
- net at T1.2 (B), T2.1 (E): now also C2.1, R2.2, R3.1
- net at T1.3 (C), T3.1 (E): now also K1.2 (B), R9.2, T10.2 (B), T8.3 (C), T9.3 (C)
- net at C1.1: now also R1.2, R2.1
- new net: C3.1, C4.1, D4.1 (K), D5.1 (K), R10.1, R11.1, R7.1, R9.1, Relé.A1
- new net: C5.1, R6.1, R7.2, R8.1
- new net: C6.1, R10.2, R12.1, T10.3 (C)
- new net: C6.2, R12.2, T11.2 (B)
- new net: T4.1 (E), T5.2 (B)
- new net: R14.2, R15.1, T4.2 (B)
- new net: D5.2 (A), R17.1, T4.3 (C), T5.3 (C)
- new net: D2.2 (A), D3.2 (A), R8.2
- new net: R4.2, R5.1, T9.2 (B)
- new net: C7.2, R16.1
- new net: D6.1 (K), R16.2, T6.2 (B)
- new net: C7.1, D4.2 (A), R11.2, R14.1, T11.3 (C)
- new net: C4.2, D1.1 (K), R4.1
- new net: R17.2, Relé.A2, T6.3 (C), T7.3 (C)
- new net: T6.1 (E), T7.2 (B)
- new net: R13.1, T10.1 (E), T11.1 (E)
- new net: R6.2, T8.2 (B)
- new net AC_power: D2.1 (K), D3.1 (K)
- new net Hangsugárzóhoz: Relé.14
Other:
- moved on the sheet: C1, C2

Commit message: vedelem
Parts:
- added C10, C11: 100nF, symbol 000_Small_Device:C
- added C8: 2200uF, symbol 000_Small_Device:C_P
- added C9: 10uF, symbol 000_Small_Device:C_P
- added D7: W01G, Diode_THT:Diode_Bridge_Round_D9.8mm, symbol Diode_Bridge:W01G
- added D8: D, symbol 000_Small_Device:D
- added U1: 7812, Converter_DCDC:Converter_DCDC_RECOM_R-78E-0.5_THT, symbol Converter_DCDC:R-7812-0.5
Connections:
- net AC_power: now also D7.2, D7.4
- net +12V0: now reaches C3.1, C4.1, D4.1 (K), D5.1 (K), R10.1, R11.1, R7.1, R9.1, Relé.A1
- net +12V0: now also C10.1, C9.1, D8.2 (A), U1.3 (OUT)
- net GNDD renamed 0V
- net 0V: now also C10.2, C11.2, C8.2, C9.2, D7.3 (-), U1.2 (GND)
- new net: C11.1, C8.1, D7.1 (+), D8.1 (K), U1.1 (IN)
Other:
- moved on the sheet: C1, C2, C3, C4, C5, C6, C7, D1, D2, D3, D4, D5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

Commit message: x
Parts:
- removed D7: W01G, Diode_THT:Diode_Bridge_Round_D9.8mm, symbol Diode_Bridge:W01G
- added D10: D8...D11: 1N...., symbol 000_Small_Device:D
- added D11, D8, D9: D, symbol 000_Small_Device:D
- added ~ (x2): (no value), symbol 000_Small_Device:Csatlakozo
- D7: renamed from D8; value D -> 1N4148
- Végfok: Érték2 Bemenete -> Kimenete
- renumbered D3 to D1, D1 to D3, R17 to R17**
Connections:
- net at C11.1, C8.1, D7.1 (K)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: now also D10.1 (K), D9.1 (K)
- net +12V0: no longer names the net of C10.1, C3.1, C4.1, C9.1, D4.1 (K), D5.1 (K), D7.2 (A), R10.1, R11.1, R7.1, R9.1, Relé.A1, U1.3 (OUT)
- net 0V renamed GNDD
- net GNDD: now also D11.2 (A), D8.2 (A)
- new net: D8.1 (K), D9.2 (A), ~.
- new net: D10.2 (A), D11.1 (K), ~.
Other:
- note added: "+"
- note added: "+11V"
- note added: "-"
- note added: "-2,2V"
- note added: "200R**"
- note added: "Hangsugárzó Védelem (Záborszky László)"
- moved on the sheet: R17**
